Commit message: adjusting the hip joints limits

File: urdf/ergoCub/robots/ergoCubGazeboV1/model.urdf (robot description, URDF)
Before this commit: robot ergoCub, 169 links, 168 joints
Joints:
- joint l_hip_roll: limit lower=-0.17453292519943295 upper=1.9547687622336491 effort=50000 velocity=120.0 -> lower=-0.34906585039 upper=1.9547687622336491 effort=50000 velocity=120.0
- joint r_hip_roll: limit lower=-0.17453292519943295 upper=1.9547687622336491 effort=50000 velocity=120.0 -> lower=-0.34906585039 upper=1.9547687622336491 effort=50000 velocity=120.0
